File: alpha.kicad_sch (KiCad schematic)
At the start: 20 parts, among them U1 ESP32-S3-PICO-1-N8R2, Y1 Crystal

Commit message: Minor edits
Parts:
- added U2: AD620, Package_SO:SOIC-8_3.9x4.9mm_P1.27mm, symbol Amplifier_Instrumentation:AD620

Commit message: More minor changes
Parts:
- added SW1: SW_Push, symbol Switch:SW_Push
Connections:
- net GND: now also SW1.1
- net at C4.2, R2.1: now also SW1.2
Other:
- note added: "A push switch here"
- note removed: "A switch here"
- moved on the sheet: C4, R2
Changed lines of the file:
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@@
 	)
 	(junction
-		(at 135.89 156.21)
-		(diameter 0)
-		(color 0 0 0 0)
-	)
-	(junction
 		(at 95.25 134.62)
 		(diameter 0)
@@
 	)
 	(junction
-		(at 111.76 162.56)
+		(at 111.76 151.13)
 		(diameter 0)
 		(color 0 0 0 0)
@@
 	)
 	(junction
+		(at 135.89 144.78)
+		(diameter 0)
+		(color 0 0 0 0)
+	)
+	(junction
 		(at 80.01 134.62)
 		(diameter 0)
@@
 	(wire
 		(pts
+			(xy 111.76 144.78) (xy 119.38 144.78)
+		)
+		(stroke
+			(width 0)
+			(type default)
+		)
+	)
+	(wire
+		(pts
 			(xy 193.04 22.86) (xy 198.12 22.86)
 		)
@@
 	(wire
 		(pts
-			(xy 111.76 156.21) (xy 111.76 162.56)
+			(xy 111.76 144.78) (xy 111.76 151.13)
 		)
 		(stroke
@@
 	(wire
 		(pts
-			(xy 135.89 156.21) (xy 143.51 156.21)
+			(xy 135.89 144.78) (xy 139.7 144.78)
 		)
 		(stroke
@@
 	(wire
 		(pts
-			(xy 135.89 162.56) (xy 135.89 156.21)
+			(xy 135.89 151.13) (xy 135.89 144.78)
 		)
 		(stroke
@@
 	(wire
 		(pts
-			(xy 128.27 162.56) (xy 135.89 162.56)
+			(xy 128.27 151.13) (xy 135.89 151.13)
 		)
 		(stroke
@@
 	(wire
 		(pts
-			(xy 203.2 87.63) (xy 203.2 97.79)
+			(xy 129.54 144.78) (xy 135.89 144.78)
 		)
 		(stroke
@@
 	(wire
 		(pts
-			(xy 100.33 52.07) (xy 77.47 52.07)
+			(xy 203.2 87.63) (xy 203.2 97.79)
 		)
 		(stroke
@@
 	(wire
 		(pts
-			(xy 68.58 100.33) (xy 68.58 97.79)
+			(xy 100.33 52.07) (xy 77.47 52.07)
 		)
 		(stroke
@@
 	(wire
 		(pts
-			(xy 111.76 156.21) (xy 120.65 156.21)
+			(xy 68.58 100.33) (xy 68.58 97.79)
 		)
 		(stroke
@@
 		)
 	)
-	(wire
-		(pts
-			(xy 151.13 156.21) (xy 158.75 156.21)
-		)
-		(stroke
-			(width 0)
-			(type default)
-		)
-	)
 	(bus
 		(pts
@@
 	(wire
 		(pts
-			(xy 111.76 162.56) (xy 111.76 165.1)
+			(xy 111.76 151.13) (xy 111.76 153.67)
 		)
 		(stroke
@@
 	(wire
 		(pts
+			(xy 147.32 144.78) (xy 151.13 144.78)
+		)
+		(stroke
+			(width 0)
+			(type default)
+		)
+	)
+	(wire
+		(pts
 			(xy 72.39 121.92) (xy 80.01 121.92)
 		)
@@
 	(wire
 		(pts
-			(xy 128.27 156.21) (xy 135.89 156.21)
-		)
-		(stroke
-			(width 0)
-			(type default)
-		)
-	)
-	(wire
-		(pts
 			(xy 95.25 121.92) (xy 102.87 121.92)
 		)
@@
 	(wire
 		(pts
-			(xy 111.76 162.56) (xy 120.65 162.56)
+			(xy 111.76 151.13) (xy 120.65 151.13)
 		)
 		(stroke
@@
 		)
 	)
-	(text "A switch here\n"
+	(text "A push switch here\n"
 		(exclude_from_sim no)
-		(at 124.46 154.94 0)
+		(at 125.222 146.812 0)
 		(effects
 			(font
@@
 		)
 	)
-	(label "EN"
-		(at 157.48 156.21 0)
-		(fields_autoplaced yes)
-		(effects
-			(font
-				(size 1.27 1.27)
-			)
-			(justify left bottom)
-		)
-	)
 	(label "1"
 		(at 213.36 92.71 0)
@@
 		)
 	)
+	(label "EN"
+		(at 151.13 144.78 0)
+		(fields_autoplaced yes)
+		(effects
+			(font
+				(size 1.27 1.27)
+			)
+			(justify left bottom)
+		)
+	)
 	(label "1"
 		(at 238.76 92.71 0)
@@
 	(symbol
 		(lib_id "Device:R")
-		(at 147.32 156.21 90)
+		(at 143.51 144.78 90)
 		(unit 1)
 		(exclude_from_sim no)
@@
 		(fields_autoplaced yes)
 		(property "Reference" "R2"
-			(at 147.32 149.86 90)
+			(at 143.51 138.43 90)
 			(effects
 				(font
@@
 		)
 		(property "Value" "R"
-			(at 147.32 152.4 90)
+			(at 143.51 140.97 90)
 			(effects
 				(font
@@
 		)
 		(property "Footprint" ""
-			(at 147.32 157.988 90)
+			(at 143.51 146.558 90)
 			(effects
 				(font
@@
 		)
 		(property "Datasheet" "~"
-			(at 147.32 156.21 0)
+			(at 143.51 144.78 0)
 			(effects
 				(font
@@
 		)
 		(property "Description" "Resistor"
-			(at 147.32 156.21 0)
+			(at 143.51 144.78 0)
 			(effects
 				(font
@@
 	(symbol
 		(lib_id "power:GND")
-		(at 111.76 165.1 0)
+		(at 111.76 153.67 0)
 		(unit 1)
 		(exclude_from_sim no)
@@
 		(fields_autoplaced yes)
 		(property "Reference" "#PWR011"
-			(at 111.76 171.45 0)
+			(at 111.76 160.02 0)
 			(effects
 				(font
@@
 		)
 		(property "Value" "GND"
-			(at 111.76 170.18 0)
+			(at 111.76 158.75 0)
 			(effects
 				(font
@@
 		)
 		(property "Footprint" ""
-			(at 111.76 165.1 0)
+			(at 111.76 153.67 0)
 			(effects
 				(font
@@
 		)
 		(property "Datasheet" ""
-			(at 111.76 165.1 0)
+			(at 111.76 153.67 0)
 			(effects
 				(font
@@
 		)
 		(property "Description" "Power symbol creates a global label with name \"GND\" , ground"
-			(at 111.76 165.1 0)
+			(at 111.76 153.67 0)
 			(effects
 				(font
@@
 	)
 	(symbol
+		(lib_id "Switch:SW_Push")
+		(at 124.46 144.78 0)
+		(unit 1)
+		(exclude_from_sim no)
+		(in_bom yes)
+		(on_board yes)
+		(dnp no)
+		(fields_autoplaced yes)
+		(property "Reference" "SW1"
+			(at 124.46 137.16 0)
+			(effects
+				(font
+					(size 1.27 1.27)
+				)
+			)
+		)
+		(property "Value" "SW_Push"
+			(at 124.46 139.7 0)
+			(effects
+				(font
+					(size 1.27 1.27)
+				)
+			)
+		)
+		(property "Footprint" ""
+			(at 124.46 139.7 0)
+			(effects
+				(font
+					(size 1.27 1.27)
+				)
+				(hide yes)
+			)
+		)
+		(property "Datasheet" "~"
+			(at 124.46 139.7 0)
+			(effects
+				(font
+					(size 1.27 1.27)
+				)
+				(hide yes)
+			)
+		)
+		(property "Description" "Push button switch, generic, two pins"
+			(at 124.46 144.78 0)
+			(effects
+				(font
+					(size 1.27 1.27)
+				)
+				(hide yes)
+			)
+		)
+		(pin "2"
+		)
+		(pin "1"
+		)
+		(instances
+			(project "alpha"
+				(path "/78da8bdf-e40e-495b-ba6c-b18ee9000176"
+					(reference "SW1")
+					(unit 1)
+				)
+			)
+		)
+	)
+	(symbol
 		(lib_id "Device:R")
 		(at 87.63 127 90)
@@
 	(symbol
 		(lib_id "Device:C")
-		(at 124.46 162.56 90)
+		(at 124.46 151.13 90)
 		(unit 1)
 		(exclude_from_sim no)
@@
 		(dnp no)
 		(property "Reference" "C4"
-			(at 124.46 170.18 90)
+			(at 124.46 158.75 90)
 			(effects
 				(font
@@
 		)
 		(property "Value" "C"
-			(at 124.46 167.64 90)
+			(at 124.46 156.21 90)
 			(effects
 				(font
@@
 		)
 		(property "Footprint" ""
-			(at 128.27 161.5948 0)
+			(at 128.27 150.1648 0)
 			(effects
 				(font
@@
 		)
 		(property "Datasheet" "~"
-			(at 124.46 162.56 0)
+			(at 124.46 151.13 0)
 			(effects
 				(font
@@
 		)
 		(property "Description" "Unpolarized capacitor"
-			(at 124.46 162.56 0)
+			(at 124.46 151.13 0)
 			(effects
 				(font

Commit message: Added Anaog Schematics
Other:
- added sheet Analog (analog.kicad_sch)
Changed lines of the file:
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@@
 	(generator "eeschema")
 	(generator_version "8.0")
-	(paper "A3")
+	(paper "A4")
 	(title_block
 		(title "Wireless ECG(ESDP 2024)")
@@
 	)
 	(bus_entry
-		(at 72.39 66.04)
+		(at 72.39 58.42)
 		(size 2.54 2.54)
 		(stroke
@@
 	)
 	(bus_entry
-		(at 69.85 66.04)
+		(at 69.85 58.42)
 		(size 2.54 2.54)
 		(stroke
@@
 	(wire
 		(pts
-			(xy 69.85 66.04) (xy 69.85 59.69)
+			(xy 69.85 58.42) (xy 69.85 52.07)
 		)
 		(stroke
@@
 	(wire
 		(pts
-			(xy 77.47 52.07) (xy 77.47 59.69)
-		)
-		(stroke
-			(width 0)
-			(type default)
-		)
-	)
-	(wire
-		(pts
 			(xy 87.63 64.77) (xy 100.33 64.77)
 		)
@@
 	(wire
 		(pts
-			(xy 72.39 59.69) (xy 72.39 66.04)
+			(xy 72.39 52.07) (xy 72.39 58.42)
 		)
 		(stroke
@@
 	(bus
 		(pts
-			(xy 69.85 68.58) (xy 72.39 68.58)
+			(xy 69.85 60.96) (xy 72.39 60.96)
 		)
 		(stroke
@@
 	(wire
 		(pts
-			(xy 77.47 59.69) (xy 72.39 59.69)
+			(xy 72.39 52.07) (xy 100.33 52.07)
 		)
 		(stroke
@@
 	(wire
 		(pts
-			(xy 100.33 52.07) (xy 77.47 52.07)
-		)
-		(stroke
-			(width 0)
-			(type default)
-		)
-	)
-	(wire
-		(pts
 			(xy 68.58 100.33) (xy 68.58 97.79)
 		)
@@
 	(bus
 		(pts
-			(xy 77.47 68.58) (xy 77.47 72.39)
+			(xy 77.47 60.96) (xy 77.47 64.77)
 		)
 		(stroke
@@
 	(wire
 		(pts
-			(xy 64.77 59.69) (xy 69.85 59.69)
+			(xy 64.77 52.07) (xy 69.85 52.07)
 		)
 		(stroke
@@
 	(bus
 		(pts
-			(xy 72.39 68.58) (xy 74.93 68.58)
+			(xy 72.39 60.96) (xy 74.93 60.96)
 		)
 		(stroke
@@
 	(bus
 		(pts
-			(xy 69.85 68.58) (xy 69.85 72.39)
+			(xy 69.85 60.96) (xy 69.85 64.77)
 		)
 		(stroke
@@
 	(bus
 		(pts
-			(xy 74.93 68.58) (xy 77.47 68.58)
+			(xy 74.93 60.96) (xy 77.47 60.96)
 		)
 		(stroke
@@
 	(bus
 		(pts
-			(xy 77.47 72.39) (xy 69.85 72.39)
+			(xy 77.47 64.77) (xy 69.85 64.77)
 		)
 		(stroke
@@
 	)
 	(label "1"
-		(at 72.39 66.04 180)
+		(at 72.39 58.42 180)
 		(fields_autoplaced yes)
 		(effects
@@
 	)
 	(label "2"
-		(at 69.85 66.04 180)
+		(at 69.85 58.42 180)
 		(fields_autoplaced yes)
 		(effects
@@
 	(symbol
 		(lib_id "power:GND")
-		(at 64.77 59.69 270)
+		(at 64.77 52.07 270)
 		(unit 1)
 		(exclude_from_sim no)
@@
 		(fields_autoplaced yes)
 		(property "Reference" "#PWR05"
-			(at 58.42 59.69 0)
+			(at 58.42 52.07 0)
 			(effects
 				(font
@@
 		)
 		(property "Value" "GND"
-			(at 60.96 59.6899 90)
+			(at 60.96 52.0699 90)
 			(effects
 				(font
@@
 		)
 		(property "Footprint" ""
-			(at 64.77 59.69 0)
+			(at 64.77 52.07 0)
 			(effects
 				(font
@@
 		)
 		(property "Datasheet" ""
-			(at 64.77 59.69 0)
+			(at 64.77 52.07 0)
 			(effects
 				(font
@@
 		)
 		(property "Description" "Power symbol creates a global label with name \"GND\" , ground"
-			(at 64.77 59.69 0)
+			(at 64.77 52.07 0)
 			(effects
 				(font
@@
 				)
 			)
+		)
+	)
+	(sheet
+		(at 19.05 16.51)
+		(size 36.83 25.4)
+		(fields_autoplaced yes)
+		(stroke
+			(width 0.1524)
+			(type solid)
+		)
+		(fill
+			(color 0 0 0 0.0000)
+		)
+		(property "Sheetname" "Analog"
+			(at 19.05 15.7984 0)
+			(effects
+				(font
+					(size 1.27 1.27)
+				)
+				(justify left bottom)
+			)
+		)
+		(property "Sheetfile" "analog.kicad_sch"
+			(at 19.05 42.4946 0)
+			(effects
+				(font
+					(size 1.27 1.27)
+				)
+				(justify left top)
+			)
+		)
+		(instances
+			(project "alpha"
+				(path "/78da8bdf-e40e-495b-ba6c-b18ee9000176"
+					(page "2")
+				)
+			)

Commit message: Revert "Added Anaog Schematics"
This reverts commit a5de0399bf14b3a200f5f1346ef0d461a1e3e6ca.
Other:
- removed sheet Analog
Changed lines of the file:
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@@
 	(generator "eeschema")
 	(generator_version "8.0")
-	(paper "A4")
+	(paper "A3")
 	(title_block
 		(title "Wireless ECG(ESDP 2024)")
@@
 	)
 	(bus_entry
-		(at 72.39 58.42)
+		(at 72.39 66.04)
 		(size 2.54 2.54)
 		(stroke
@@
 	)
 	(bus_entry
-		(at 69.85 58.42)
+		(at 69.85 66.04)
 		(size 2.54 2.54)
 		(stroke
@@
 	(wire
 		(pts
-			(xy 69.85 58.42) (xy 69.85 52.07)
+			(xy 69.85 66.04) (xy 69.85 59.69)
 		)
 		(stroke
@@
 	(wire
 		(pts
+			(xy 77.47 52.07) (xy 77.47 59.69)
+		)
+		(stroke
+			(width 0)
+			(type default)
+		)
+	)
+	(wire
+		(pts
 			(xy 87.63 64.77) (xy 100.33 64.77)
 		)
@@
 	(wire
 		(pts
-			(xy 72.39 52.07) (xy 72.39 58.42)
+			(xy 72.39 59.69) (xy 72.39 66.04)
 		)
 		(stroke
@@
 	(bus
 		(pts
-			(xy 69.85 60.96) (xy 72.39 60.96)
+			(xy 69.85 68.58) (xy 72.39 68.58)
 		)
 		(stroke
@@
 	(wire
 		(pts
-			(xy 72.39 52.07) (xy 100.33 52.07)
+			(xy 77.47 59.69) (xy 72.39 59.69)
 		)
 		(stroke
@@
 	(wire
 		(pts
+			(xy 100.33 52.07) (xy 77.47 52.07)
+		)
+		(stroke
+			(width 0)
+			(type default)
+		)
+	)
+	(wire
+		(pts
 			(xy 68.58 100.33) (xy 68.58 97.79)
 		)
@@
 	(bus
 		(pts
-			(xy 77.47 60.96) (xy 77.47 64.77)
+			(xy 77.47 68.58) (xy 77.47 72.39)
 		)
 		(stroke
@@
 	(wire
 		(pts
-			(xy 64.77 52.07) (xy 69.85 52.07)
+			(xy 64.77 59.69) (xy 69.85 59.69)
 		)
 		(stroke
@@
 	(bus
 		(pts
-			(xy 72.39 60.96) (xy 74.93 60.96)
+			(xy 72.39 68.58) (xy 74.93 68.58)
 		)
 		(stroke
@@
 	(bus
 		(pts
-			(xy 69.85 60.96) (xy 69.85 64.77)
+			(xy 69.85 68.58) (xy 69.85 72.39)
 		)
 		(stroke
@@
 	(bus
 		(pts
-			(xy 74.93 60.96) (xy 77.47 60.96)
+			(xy 74.93 68.58) (xy 77.47 68.58)
 		)
 		(stroke
@@
 	(bus
 		(pts
-			(xy 77.47 64.77) (xy 69.85 64.77)
+			(xy 77.47 72.39) (xy 69.85 72.39)
 		)
 		(stroke
@@
 	)
 	(label "1"
-		(at 72.39 58.42 180)
+		(at 72.39 66.04 180)
 		(fields_autoplaced yes)
 		(effects
@@
 	)
 	(label "2"
-		(at 69.85 58.42 180)
+		(at 69.85 66.04 180)
 		(fields_autoplaced yes)
 		(effects
@@
 	(symbol
 		(lib_id "power:GND")
-		(at 64.77 52.07 270)
+		(at 64.77 59.69 270)
 		(unit 1)
 		(exclude_from_sim no)
@@
 		(fields_autoplaced yes)
 		(property "Reference" "#PWR05"
-			(at 58.42 52.07 0)
+			(at 58.42 59.69 0)
 			(effects
 				(font
@@
 		)
 		(property "Value" "GND"
-			(at 60.96 52.0699 90)
+			(at 60.96 59.6899 90)
 			(effects
 				(font
@@
 		)
 		(property "Footprint" ""
-			(at 64.77 52.07 0)
+			(at 64.77 59.69 0)
 			(effects
 				(font
@@
 		)
 		(property "Datasheet" ""
-			(at 64.77 52.07 0)
+			(at 64.77 59.69 0)
 			(effects
 				(font
@@
 		)
 		(property "Description" "Power symbol creates a global label with name \"GND\" , ground"
-			(at 64.77 52.07 0)
+			(at 64.77 59.69 0)
 			(effects
 				(font
@@
 				)
 			)
-		)
-	)
-	(sheet
-		(at 19.05 16.51)
-		(size 36.83 25.4)
-		(fields_autoplaced yes)
-		(stroke
-			(width 0.1524)
-			(type solid)
-		)
-		(fill
-			(color 0 0 0 0.0000)
-		)
-		(property "Sheetname" "Analog"
-			(at 19.05 15.7984 0)
-			(effects
-				(font
-					(size 1.27 1.27)
-				)
-				(justify left bottom)
-			)
-		)
-		(property "Sheetfile" "analog.kicad_sch"
-			(at 19.05 42.4946 0)
-			(effects
-				(font
-					(size 1.27 1.27)
-				)
-				(justify left top)
-			)
-		)
-		(instances
-			(project "alpha"
-				(path "/78da8bdf-e40e-495b-ba6c-b18ee9000176"
-					(page "2")
-				)
-			)
